Commit message: modify info.py and teach_mode first edition

File: universal_robot/ur_description/urdf/ur5.urdf.xacro (robot description, xacro)
@@ -127,5 +127,5 @@
       </xacro:unless>
       <xacro:if value="${joint_limited}">
-        <limit lower="${-pi}" upper="${pi}" effort="150.0" velocity="3.15"/>
+        <limit lower="${-pi}" upper="0.0" effort="150.0" velocity="3.15"/>
       </xacro:if>
       <dynamics damping="0.0" friction="0.0"/>

File: universal_robot/ur_description/urdf/ur5_joint_limited_robot.urdf.xacro (robot description, xacro)
@@ -8,48 +8,9 @@
   <!-- arm -->
   <xacro:ur5_robot prefix="" joint_limited="true"/>
-  <!-- gazebo material-->
-  <xacro:include filename="$(find ur_description)/urdf/ur5.gazebo" />
-  <xacro:include filename="$(find ur_description)/urdf/materials.xacro" />
-  <!-- param-->
-  <xacro:property name="width" value="0.1" /> <!-- Square dimensions (widthxwidth) of beams -->
-  <xacro:property name="height1" value="0.9" /> <!-- Link 1       <material name="orange"/> -->
   <link name="world" />
-  <!--joint name="world_joint" type="fixed">
+  <joint name="world_joint" type="fixed">
     <parent link="world" />
     <child link = "base_link" />
     <origin xyz="0.0 0.0 0.0" rpy="0.0 0.0 0.0" />
-  </joint-->
-  <joint name="world_joint" type="fixed">
-    <parent link="world" />
-    <child link = "link1" />
-    <origin xyz="0.0 0.0 0.0" rpy="0.0 0.0 0.0" />
-  </joint>
-  <link name="link1">
-    <collision>
-      <origin xyz="-0.6 -0.6 0.0" rpy="0 0 0"/>
-      <geometry>
-	<mesh filename="package://ur_description/meshes/ur5/collision/column.stl" scale="0.001 0.001 0.001"/>
-      </geometry>
-    </collision>
-    <visual>
-      <origin xyz="-0.6 -0.6 0.0" rpy="0 0 0"/>
-      <geometry>
-	<mesh filename="package://ur_description/meshes/ur5/collision/column.stl" scale="0.001 0.001 0.001"/>
-      </geometry>
-      <material name="orange"/>
-    </visual>
-    <inertial>
-      <origin xyz="-0.6 -0.6 0.0" rpy="0 0 0"/>
-      <mass value="1"/>
-      <inertia
-	  ixx="1.0" ixy="0.0" ixz="0.0"
-	  iyy="1.0" iyz="0.0"
-	  izz="1.0"/>
-    </inertial>
-  </link>
-  <joint name="link1_joint" type="fixed">
-    <parent link="link1" />
-    <child link = "base_link" />
-    <origin xyz="0.0 0.0 ${height1}" rpy="0.0 0.0 0.0" />
   </joint>
 </robot>

Commit message: Add column and vaccum in to ur_description

File: universal_robot/ur_description/urdf/ur5.urdf.xacro (robot description, xacro)
@@ -127,5 +127,5 @@
       </xacro:unless>
       <xacro:if value="${joint_limited}">
-        <limit lower="${-pi}" upper="0.0" effort="150.0" velocity="3.15"/>
+        <limit lower="${-pi}" upper="${pi}" effort="150.0" velocity="3.15"/>
       </xacro:if>
       <dynamics damping="0.0" friction="0.0"/>
@@ -280,8 +280,30 @@
     <link name="${prefix}ee_link">
       <collision>
+        <origin xyz="0.04 0.1 0.0" rpy="0 0 0"/>
+        <geometry>
+          <box size="0.08 0.3 0.10"/>
+        </geometry>
+      </collision>
+      <visual>
+        <origin xyz="0.1 -0.05 -0.04" rpy="0 -1.57 0"/>
+        <geometry>
+          <mesh filename="package://ur_description/meshes/ur5/visual/ur5_tmp_vaccum.STL" scale="0.001 0.001 0.001"/>
+        </geometry>
+        <material name="orange">
+          <color rgba="0.7 0.7 0.7 1.0"/>
+        </material>
+      </visual>
+    </link>
+    <joint name="$vaccum_joint" type="fixed">
+      <parent link="${prefix}ee_link" />
+      <child link = "${prefix}vaccum_link" />
+      <origin xyz="0.1 0.23 0.0" rpy="0.0 0.0 0.0" />
+    </joint>
+    <link name="${prefix}vaccum_link">
+      <collision>
         <geometry>
           <box size="0.01 0.01 0.01"/>
         </geometry>
-        <origin rpy="0 0 0" xyz="-0.01 0 0"/>
+        <origin rpy="0 0 0" xyz="0.0 0 0"/>
       </collision>
     </link>

File: universal_robot/ur_description/urdf/ur5_joint_limited_robot.urdf.xacro (robot description, xacro)
@@ -8,9 +8,48 @@
   <!-- arm -->
   <xacro:ur5_robot prefix="" joint_limited="true"/>
+  <!-- gazebo material-->
+  <xacro:include filename="$(find ur_description)/urdf/ur5.gazebo" />
+  <xacro:include filename="$(find ur_description)/urdf/materials.xacro" />
+  <!-- param-->
+  <xacro:property name="width" value="0.1" /> <!-- Square dimensions (widthxwidth) of beams -->
+  <xacro:property name="height1" value="0.9" /> <!-- Link 1       <material name="orange"/> -->
   <link name="world" />
-  <joint name="world_joint" type="fixed">
+  <!--joint name="world_joint" type="fixed">
     <parent link="world" />
     <child link = "base_link" />
     <origin xyz="0.0 0.0 0.0" rpy="0.0 0.0 0.0" />
+  </joint-->
+  <joint name="world_joint" type="fixed">
+    <parent link="world" />
+    <child link = "link1" />
+    <origin xyz="0.0 0.0 0.0" rpy="0.0 0.0 0.0" />
+  </joint>
+  <link name="link1">
+    <collision>
+      <origin xyz="0.0 0.0 0.45" rpy="0 0 0"/>
+      <geometry>
+	<box size="0.1 0.1 0.9"/>
+      </geometry>
+    </collision>
+    <visual>
+      <origin xyz="-0.6 -0.6 0.0" rpy="0 0 0"/>
+      <geometry>
+	<mesh filename="package://ur_description/meshes/ur5/visual/column.stl" scale="0.001 0.001 0.001"/>
+      </geometry>
+      <material name="gray"/>
+    </visual>
+    <inertial>
+      <origin xyz="-0.6 -0.6 0.0" rpy="0 0 0"/>
+      <mass value="1"/>
+      <inertia
+	  ixx="1.0" ixy="0.0" ixz="0.0"
+	  iyy="1.0" iyz="0.0"
+	  izz="1.0"/>
+    </inertial>
+  </link>
+  <joint name="link1_joint" type="fixed">
+    <parent link="link1" />
+    <child link = "base_link" />
+    <origin xyz="0.0 0.0 ${height1}" rpy="0.0 0.0 0.0" />
   </joint>
 </robot>

Commit message: Modify some urdf:eef and srdf:eef

File: universal_robot/ur_description/urdf/ur5.urdf.xacro (robot description, xacro)
@@ -276,5 +276,5 @@
       <parent link="${prefix}wrist_3_link" />
       <child link = "${prefix}ee_link" />
-      <origin xyz="0.0 ${wrist_3_length} 0.0" rpy="0.0 0.0 ${pi/2.0}" />
+      <origin xyz="0.0 ${wrist_3_length} 0.0" rpy="${pi/2.0} 0.0 ${pi/2.0}" />
     </joint>
     <link name="${prefix}ee_link">
